File: 005k/pcb/pcb.kicad_pcb (KiCad board)
At the start: 2 copper layers, 295.5 x 108.4 mm, 105 parts, among them U1 ProMicro

Commit message: dim. 10 déc. 2023 12:03:13 CET
Parts:
- removed D48: 1N4148, Diode_THT:D_DO-35_SOD27_P7.62mm_Horizontal
- removed MX48: MX, mx:MX-Alps-Hybrid-1U
- removed REF01, REF02, REF03, REF04, REF05, REF06, REF07, REF08, REF09: MountingHole_2.2mm_M2, MountingHole:MountingHole_2.2mm_M2
- added D22: 1N4148, Diode_THT:D_DO-35_SOD27_P7.62mm_Horizontal, F.Cu at (283.6, 130.9)
- added J1: Screw_Terminal_01x04, oled:SSD1306-0.91-OLED-4pin-128x32, F.Cu at (209.1, 124.6)
- added MX22: MX, mx:MX-Alps-Hybrid-1U, F.Cu at (285.9, 122.3)
- added REF1: MountingHole_2.2mm_M2, MountingHole:MountingHole_2.2mm_M2, F.Cu at (233.2, 106.4)
- added REF11: MountingHole_2.2mm_M2, MountingHole:MountingHole_2.2mm_M2, F.Cu at (203.2, 167.4)
- added REF2: MountingHole_2.2mm_M2, MountingHole:MountingHole_2.2mm_M2, F.Cu at (273.2, 95.4)
- added REF3: MountingHole_2.2mm_M2, MountingHole:MountingHole_2.2mm_M2, F.Cu at (344.8, 171.8)
- added REF4: MountingHole_2.2mm_M2, MountingHole:MountingHole_2.2mm_M2, F.Cu at (277.2, 158.4)
- added REF5: MountingHole_2.2mm_M2, MountingHole:MountingHole_2.2mm_M2, F.Cu at (256.3, 187.4)
- added REF6: MountingHole_2.2mm_M2, MountingHole:MountingHole_2.2mm_M2, F.Cu at (150.1, 187.4)
- added REF7: MountingHole_2.2mm_M2, MountingHole:MountingHole_2.2mm_M2, F.Cu at (129.2, 158.4)
- added REF8: MountingHole_2.2mm_M2, MountingHole:MountingHole_2.2mm_M2, F.Cu at (61.6, 171.8)
- added REF9: MountingHole_2.2mm_M2, MountingHole:MountingHole_2.2mm_M2, F.Cu at (133.2, 95.4)
- MX1, MX25: footprint mx:MX-Alps-Hybrid-1.25U -> mx:MX-Alps-Hybrid-1U
- MX24: footprint mx:MX-Alps-Hybrid-2.75U -> mx:MX-Alps-Hybrid-1U
- MX31, MX7: footprint mx:MX-Alps-Hybrid-1.75U -> mx:MX-Alps-Hybrid-1U
- moved D37 250.6 mm to (67.2, 169.4), turned to -10 degrees
- moved MX37 248.0 mm to (72.3, 162.2), turned to -10 degrees
- moved D25 244.9 mm to (70.5, 150.7), turned to -10 degrees
- moved MX25 242.4 mm to (75.6, 143.4), turned to -10 degrees
- moved D38 210.4 mm to (88.3, 173.1), turned to -10 degrees
- moved MX38 207.8 mm to (93.4, 165.9), turned to -10 degrees
- moved D26 201.5 mm to (92.4, 149.7), turned to -10 degrees
- moved MX26 199.0 mm to (97.6, 142.5), turned to -10 degrees
- moved D39 170.6 mm to (109.4, 176.9), turned to -10 degrees
- moved MX39 168.0 mm to (114.5, 169.6), turned to -10 degrees
- moved D27 163.0 mm to (112.0, 148.3), turned to -10 degrees
- moved MX27 160.6 mm to (117.2, 141.1), turned to -10 degrees
- moved D19 159.2 mm to (228.1, 145.5), turned to 10 degrees
- moved D23 157.3 mm to (303.2, 132.3), turned to 10 degrees
- moved MX19 156.7 mm to (230.5, 136.9), turned to 10 degrees
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Connections:
- D10 pad 1: L2 -> L5
- D11 pad 1: L2 -> L5
- D12 pad 1: L2 -> L5
- D13 pad 1: L3 -> L2
- D14 pad 1: L3 -> L2
- D15 pad 1: L3 -> L2
- D16 pad 1: L3 -> L2
- D17 pad 1: L3 -> L2
- D18 pad 1: L3 -> L2
- D19 pad 1: L4 -> L6
- D20 pad 1: L4 -> L6
- D21 pad 1: L4 -> L6
- D23 pad 1: L4 -> L6
- D24 pad 1: L4 -> L6
- D25 pad 1: L5 -> L3
- D26 pad 1: L5 -> L3
- D27 pad 1: L5 -> L3
- D28 pad 1: L5 -> L3
- D29 pad 1: L5 -> L3
- D30 pad 1: L5 -> L3
- D31 pad 1: L6 -> L7
- D32 pad 1: L6 -> L7
- D33 pad 1: L6 -> L7
- D34 pad 1: L6 -> L7
- D35 pad 1: L6 -> L7
- D36 pad 1: L6 -> L7
- D37 pad 1: L7 -> L4
- D38 pad 1: L7 -> L4
- D39 pad 1: L7 -> L4
- D40 pad 1: L7 -> L4
- D41 pad 1: L7 -> L4
- D42 pad 1: L7 -> L8
- D7 pad 1: L2 -> L5
- D8 pad 1: L2 -> L5
- D9 pad 1: L2 -> L5
- MX10 pad 1: C4 -> C3
- MX11 pad 1: C5 -> C2
- MX12 pad 1: C6 -> C1
- MX19 pad 1: C1 -> C6
- MX20 pad 1: C2 -> C5
- MX21 pad 1: C3 -> C4
- MX23 pad 1: C5 -> C2
- MX24 pad 1: C6 -> C1
- MX31 pad 1: C1 -> C6
- MX32 pad 1: C2 -> C5
- MX33 pad 1: C3 -> C4
- MX34 pad 1: C4 -> C3
- MX35 pad 1: C5 -> C2
- MX36 pad 1: C6 -> C1
- MX40 pad 1: C4 -> C5
- MX41 pad 1: C5 -> C6
- MX43 pad 1: C1 -> C5
- MX44 pad 1: C2 -> C4
- MX46 pad 1: C4 -> C2
- MX47 pad 1: C5 -> C1
- MX7 pad 1: C1 -> C6
- MX8 pad 1: C2 -> C5
- MX9 pad 1: C3 -> C4
- U1 pad 14: unconnected-(U1-GND-Pad14) -> GND
- U1 pad 16: unconnected-(U1-VCC-Pad16) -> VCC
- U1 pad 17: unconnected-(U1-F4-Pad17) -> C6
- U1 pad 18: C4 -> C5
- U1 pad 19: C5 -> C4
- U1 pad 20: C6 -> C3
- U1 pad 3: unconnected-(U1-GND-Pad3) -> GND
- U1 pad 4: unconnected-(U1-GND-Pad4) -> GND
- U1 pad 5: unconnected-(U1-D1-Pad5) -> SDA
- U1 pad 6: C1 -> SCL
- U1 pad 8: C3 -> C1
Routing:
- net C2: track 0.00 -> 446.3 mm, vias 0 -> 1
- net C1: track 0.00 -> 434.0 mm, vias 0 -> 1
- net C3: track 0.00 -> 421.4 mm, vias 0 -> 1
- net C4: track 0.00 -> 335.0 mm, vias 0 -> 1
- net C5: track 0.00 -> 288.6 mm, vias 0 -> 1
- net C6: track 0.00 -> 230.7 mm
- net L8: track 0.00 -> 212.7 mm
- net L4: track 0.00 -> 187.1 mm
- net L3: track 0.00 -> 164.8 mm
- net L1: track 0.00 -> 160.8 mm
- net L7: track 0.00 -> 156.3 mm
- net L2: track 0.00 -> 149.4 mm
- net L5: track 0.00 -> 146.0 mm
- net L6: track 0.00 -> 140.2 mm
- net GND: track 0.00 -> 47.4 mm
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- added copper zone on B.Cu, net GND
- added copper zone on F.Cu, net GND
Other:
- board size 295.5 x 108.4 mm -> 293.2 x 106 mm

Commit message: dim. 10 déc. 2023 13:12:07 CET
Routing:
- net C6: track 230.7 -> 220.3 mm
- net C1: track 434.0 -> 424.4 mm
- net C3: track 421.4 -> 430.0 mm
- net C5: track 288.6 -> 294.3 mm
- net C2: track 446.3 -> 443.9 mm, vias 1 -> 0
- net C4: track 335.0 -> 337.2 mm
- net L6: track 140.2 -> 138.2 mm
- net L1: track 160.8 -> 159.2 mm
- net L7: track 156.3 -> 155.0 mm

Commit message: dim. 10 déc. 2023 20:23:19 CET
Parts:
- MX1, MX12, MX13, MX24, MX25, MX36, MX37, MX39, MX40, MX41, MX43, MX44: footprint mx:MX-Alps-Hybrid-1U -> mx:MX-Alps-Hybrid-1.25U
- MX42: footprint mx:MX-Alps-Hybrid-1U -> mx:MX-Alps-Hybrid-2.25U
Routing:
- net C6: track 220.3 -> 226.6 mm
- net C3: track 430.0 -> 424.0 mm
- net L8: track 212.6 -> 208.1 mm
- net C4: track 337.2 -> 333.5 mm
- net L4: track 187.1 -> 185.6 mm
- net C2: track 443.9 -> 442.4 mm
- net L1: track 159.2 -> 158.3 mm
