File: 005k/pcb/pcb.kicad_pcb (KiCad board)
At the start: 2 copper layers, 293.2 x 106 mm, 107 parts, among them J1 Screw_Terminal_01x04, U1 ProMicro

Commit message: jeu. 28 déc. 2023 20:04:29 CET
Parts:
- removed D47: 1N4148, Diode_THT:D_DO-35_SOD27_P7.62mm_Horizontal
- removed MX47: MX, mx:MX-Alps-Hybrid-1U
- removed REF1, REF10, REF11, REF2, REF3, REF4, REF5, REF6, REF7, REF8, REF9: MountingHole_2.2mm_M2, MountingHole:MountingHole_2.2mm_M2
- added J101: Screw_Terminal_01x01, MountingHole:MountingHole_2.2mm_M2, F.Cu at (116.2, 112.3)
- added J102: Screw_Terminal_01x01, MountingHole:MountingHole_2.2mm_M2, F.Cu at (83.6, 150.1)
- added J103: Screw_Terminal_01x01, MountingHole:MountingHole_2.2mm_M2, F.Cu at (237.4, 125.5)
- added J104: Screw_Terminal_01x01, MountingHole:MountingHole_2.2mm_M2, F.Cu at (345.0, 150.1)
- added J105: Screw_Terminal_01x01, MountingHole:MountingHole_2.2mm_M2, F.Cu at (241.2, 186.1)
- added J106: Screw_Terminal_01x01, MountingHole:MountingHole_2.2mm_M2, F.Cu at (191.2, 125.5)
- added J107: Screw_Terminal_01x01, MountingHole:MountingHole_2.2mm_M2, F.Cu at (128.3, 153.1)
- added J108: Screw_Terminal_01x01, MountingHole:MountingHole_2.2mm_M2, F.Cu at (300.3, 153.1)
- added J109: Screw_Terminal_01x01, MountingHole:MountingHole_2.2mm_M2, F.Cu at (312.4, 112.3)
- added J110: Screw_Terminal_01x01, MountingHole:MountingHole_2.2mm_M2, F.Cu at (187.5, 186.1)
- J1: value Screw_Terminal_01x04 -> Conn_01x04_Socket; footprint oled:SSD1306-0.91-OLED-4pin-128x32 -> _OLED:SSD1306-0.91-OLED-4pin-128x32
- MX1, MX12, MX13, MX24, MX25, MX36, MX37, MX39, MX40: footprint mx:MX-Alps-Hybrid-1.25U -> _mx:MX-Alps-Hybrid-1.25U
- MX10, MX11, MX14, MX15, MX16, MX17, MX18, MX19, MX2, MX20, MX21, MX22, MX23, MX26, MX27, MX28, MX29, MX3, MX30, MX31, MX32, MX33, MX34, MX35, MX4, MX45, MX46, MX5, MX6, MX7, MX8, MX9: footprint mx:MX-Alps-Hybrid-1U -> _mx:MX-Alps-Hybrid-1U
- MX38: footprint mx:MX-Alps-Hybrid-1U -> _mx:MX-Alps-Hybrid-1.25U
- MX41: footprint mx:MX-Alps-Hybrid-1.25U -> _mx:MX-Alps-Hybrid-3U-ReversedStabilizers
- MX42: footprint mx:MX-Alps-Hybrid-2.25U -> _mx:MX-Alps-Hybrid-1.25U
- MX43, MX44: footprint mx:MX-Alps-Hybrid-1.25U -> _mx:MX-Alps-Hybrid-1U
- moved D42 70.6 mm to (269.7, 180.0), turned to 90 degrees
- moved MX43 63.8 mm to (302.8, 167.2)
- moved D43 58.6 mm to (294.0, 172.6), turned to 100 degrees
- moved D41 57.6 mm to (210.5, 162.6), turned to 0 degrees
- moved MX42 56.7 mm to (259.6, 176.2)
- moved MX44 54.3 mm to (321.5, 163.9)
- moved MX41 49.1 mm to (214.3, 181.0), turned to 0 degrees
- moved D44 48.8 mm to (312.8, 169.3), turned to 100 degrees
- moved MX45 46.9 mm to (340.3, 160.6)
- moved D45 41.4 mm to (331.6, 166.0), turned to 100 degrees
- moved D39 37.0 mm to (146.3, 174.7), turned to 80 degrees
- moved D38 34.7 mm to (122.9, 170.5), turned to 80 degrees
- moved MX46 32.8 mm to (281.5, 156.4)
- moved D37 32.4 mm to (99.4, 166.4), turned to 80 degrees
- moved MX40 32.0 mm to (169.1, 176.2), turned to 0 degrees
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Connections:
- MX42 pad 1: C6 -> C5
- MX43 pad 1: C5 -> C3
- MX44 pad 1: C4 -> C2
- MX45 pad 1: C3 -> C1
- MX46 pad 1: C2 -> C4
- U1 pad 17: C6 -> C3
- U1 pad 18: C5 -> C4
- U1 pad 19: C4 -> C5
- U1 pad 20: C3 -> C6
- U1 pad 7: C2 -> C1
- U1 pad 8: C1 -> C2
Routing:
- net C1: track 424.4 -> 553.8 mm, vias 1 -> 0
- net C4: track 333.5 -> 252.7 mm, vias 1 -> 0
- net L8: track 208.1 -> 153.8 mm
- net C3: track 424.0 -> 374.7 mm, vias 1 -> 0
- net GND: track 47.4 -> 0.00 mm
- net C6: track 226.6 -> 181.0 mm
- net L4: track 185.6 -> 142.9 mm
- net C5: track 294.3 -> 259.3 mm, vias 1 -> 0
- net L3: track 164.8 -> 130.0 mm
- net C2: track 442.4 -> 473.4 mm
- net L2: track 149.4 -> 123.8 mm
- net L1: track 158.3 -> 141.3 mm
- net L7: track 155.0 -> 138.8 mm
- net L6: track 138.2 -> 124.0 mm
- net Net-(D47-A): track 13.5 -> 0.00 mm
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Other:
- board size 293.2 x 106 mm -> 279.9 x 110.1 mm

Commit message: jeu. 28 déc. 2023 23:03:25 CET
Parts:
- MX41: footprint _mx:MX-Alps-Hybrid-3U-ReversedStabilizers -> _mx:MX-Alps-Hybrid-2.75U-ReversedStabilizers
Routing:
- net C6: track 181.0 -> 185.1 mm
- net L4: track 142.9 -> 139.2 mm

Commit message: ven. 29 déc. 2023 11:31:16 CET
Routing:
- net C2: track 473.4 -> 472.6 mm
