File: 005k/pcb/pcb.kicad_sch (KiCad schematic)
At the start: 96 parts, among them J1 Screw_Terminal_01x04, U1 ProMicro

Commit message: dim. 10 déc. 2023 20:23:19 CET
Parts:
- MX1, MX12, MX13, MX24, MX25, MX36, MX37, MX39, MX40, MX41, MX43, MX44: footprint mx:MX-Alps-Hybrid-1U -> mx:MX-Alps-Hybrid-1.25U
- MX42: footprint mx:MX-Alps-Hybrid-1U -> mx:MX-Alps-Hybrid-2.25U
Changed lines of the file:
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@@
       (effects (font (size 0.508 0.508)) hide)
     )
-    (property "Footprint" "mx:MX-Alps-Hybrid-1U" (at 176.53 101.6 0)
+    (property "Footprint" "mx:MX-Alps-Hybrid-2.25U" (at 176.53 101.6 0)
       (effects (font (size 1.27 1.27)) hide)
     )
@@
       (effects (font (size 0.508 0.508)) hide)
     )
-    (property "Footprint" "mx:MX-Alps-Hybrid-1U" (at 154.94 101.6 0)
+    (property "Footprint" "mx:MX-Alps-Hybrid-1.25U" (at 154.94 101.6 0)
       (effects (font (size 1.27 1.27)) hide)
     )
@@
       (effects (font (size 0.508 0.508)) hide)
     )
-    (property "Footprint" "mx:MX-Alps-Hybrid-1U" (at 104.14 55.88 0)
+    (property "Footprint" "mx:MX-Alps-Hybrid-1.25U" (at 104.14 55.88 0)
       (effects (font (size 1.27 1.27)) hide)
     )
@@
       (effects (font (size 0.508 0.508)) hide)
     )
-    (property "Footprint" "mx:MX-Alps-Hybrid-1U" (at 227.33 55.88 0)
+    (property "Footprint" "mx:MX-Alps-Hybrid-1.25U" (at 227.33 55.88 0)
       (effects (font (size 1.27 1.27)) hide)
     )
@@
       (effects (font (size 0.508 0.508)) hide)
     )
-    (property "Footprint" "mx:MX-Alps-Hybrid-1U" (at 144.78 101.6 0)
+    (property "Footprint" "mx:MX-Alps-Hybrid-1.25U" (at 144.78 101.6 0)
       (effects (font (size 1.27 1.27)) hide)
     )
@@
       (effects (font (size 0.508 0.508)) hide)
     )
-    (property "Footprint" "mx:MX-Alps-Hybrid-1U" (at 124.46 101.6 0)
+    (property "Footprint" "mx:MX-Alps-Hybrid-1.25U" (at 124.46 101.6 0)
       (effects (font (size 1.27 1.27)) hide)
     )
@@
       (effects (font (size 0.508 0.508)) hide)
     )
-    (property "Footprint" "mx:MX-Alps-Hybrid-1U" (at 196.85 101.6 0)
+    (property "Footprint" "mx:MX-Alps-Hybrid-1.25U" (at 196.85 101.6 0)
       (effects (font (size 1.27 1.27)) hide)
     )
@@
       (effects (font (size 0.508 0.508)) hide)
     )
-    (property "Footprint" "mx:MX-Alps-Hybrid-1U" (at 104.14 33.02 0)
+    (property "Footprint" "mx:MX-Alps-Hybrid-1.25U" (at 104.14 33.02 0)
       (effects (font (size 1.27 1.27)) hide)
     )
@@
       (effects (font (size 0.508 0.508)) hide)
     )
-    (property "Footprint" "mx:MX-Alps-Hybrid-1U" (at 227.33 78.74 0)
+    (property "Footprint" "mx:MX-Alps-Hybrid-1.25U" (at 227.33 78.74 0)
       (effects (font (size 1.27 1.27)) hide)
     )
@@
       (effects (font (size 0.508 0.508)) hide)
     )
-    (property "Footprint" "mx:MX-Alps-Hybrid-1U" (at 227.33 33.02 0)
+    (property "Footprint" "mx:MX-Alps-Hybrid-1.25U" (at 227.33 33.02 0)
       (effects (font (size 1.27 1.27)) hide)
     )
@@
       (effects (font (size 0.508 0.508)) hide)
     )
-    (property "Footprint" "mx:MX-Alps-Hybrid-1U" (at 104.14 78.74 0)
+    (property "Footprint" "mx:MX-Alps-Hybrid-1.25U" (at 104.14 78.74 0)
       (effects (font (size 1.27 1.27)) hide)
     )
@@
       (effects (font (size 0.508 0.508)) hide)
     )
-    (property "Footprint" "mx:MX-Alps-Hybrid-1U" (at 104.14 101.6 0)
+    (property "Footprint" "mx:MX-Alps-Hybrid-1.25U" (at 104.14 101.6 0)
       (effects (font (size 1.27 1.27)) hide)
     )
@@
       (effects (font (size 0.508 0.508)) hide)
     )
-    (property "Footprint" "mx:MX-Alps-Hybrid-1U" (at 186.69 101.6 0)
-      (effects (font (size 1.27 1.27)) hide)
-    )
+    (property "Footprint" "mx:MX-Alps-Hybrid-1.25U" (at 186.69 101.6 0)
+      (effects (font (size 1.27 1.27)) hide)
+    )

Commit message: jeu. 28 déc. 2023 20:04:29 CET
Parts:
- removed D47: 1N4148, Diode_THT:D_DO-35_SOD27_P7.62mm_Horizontal, symbol Diode:1N4148
- removed J1: Screw_Terminal_01x04, oled:SSD1306-0.91-OLED-4pin-128x32, symbol Connector:Screw_Terminal_01x04
- removed MX47: MX, mx:MX-Alps-Hybrid-1U, symbol PCM_0xcb:MX
- added J1: Conn_01x04_Socket, _OLED:SSD1306-0.91-OLED-4pin-128x32, symbol Connector:Conn_01x04_Socket
- added J101, J102, J103, J104, J105, J106, J107, J108, J109, J110: Screw_Terminal_01x01, MountingHole:MountingHole_2.2mm_M2, symbol Connector:Screw_Terminal_01x01
- MX1, MX12, MX13, MX24, MX25, MX36, MX37, MX39, MX40: footprint mx:MX-Alps-Hybrid-1.25U -> _mx:MX-Alps-Hybrid-1.25U
- MX10, MX11, MX14, MX15, MX16, MX17, MX18, MX19, MX2, MX20, MX21, MX22, MX23, MX26, MX27, MX28, MX29, MX3, MX30, MX31, MX32, MX33, MX34, MX35, MX4, MX45, MX46, MX5, MX6, MX7, MX8, MX9: footprint mx:MX-Alps-Hybrid-1U -> _mx:MX-Alps-Hybrid-1U
- MX38: footprint mx:MX-Alps-Hybrid-1U -> _mx:MX-Alps-Hybrid-1.25U
- MX41: footprint mx:MX-Alps-Hybrid-1.25U -> _mx:MX-Alps-Hybrid-3U-ReversedStabilizers
- MX42: footprint mx:MX-Alps-Hybrid-2.25U -> _mx:MX-Alps-Hybrid-1.25U
- MX43, MX44: footprint mx:MX-Alps-Hybrid-1.25U -> _mx:MX-Alps-Hybrid-1U
Connections:
- net C1: now also MX45.1 (COL), U1.7 (D4); no longer U1.8 (C6)
- net C2: now also MX44.1 (COL), U1.8 (C6); no longer MX46.1 (COL), U1.7 (D4)
- net C3: now also MX43.1 (COL), U1.17 (F4); no longer MX45.1 (COL), U1.20 (F7)
- net C4: now also MX46.1 (COL), U1.18 (F5); no longer MX44.1 (COL), U1.19 (F6)
- net C5: now also MX42.1 (COL), U1.19 (F6); no longer MX43.1 (COL), U1.18 (F5)
- net C6: now also U1.20 (F7); no longer MX42.1 (COL), U1.17 (F4)
- net GND: now also J1.1 (Pin_1), J101.1 (Pin_1), J102.1 (Pin_1), J103.1 (Pin_1), J104.1 (Pin_1), J105.1 (Pin_1), J106.1 (Pin_1), J107.1 (Pin_1), J108.1 (Pin_1), J109.1 (Pin_1), J110.1 (Pin_1)
- net SCL: now also J1.3 (Pin_3)
- net SDA: now also J1.4 (Pin_4)
- net VCC: now also J1.2 (Pin_2)

Commit message: jeu. 28 déc. 2023 23:03:25 CET
Parts:
- MX41: footprint _mx:MX-Alps-Hybrid-3U-ReversedStabilizers -> _mx:MX-Alps-Hybrid-2.75U-ReversedStabilizers
