File: 007k/pcb/little/_autosave-little.kicad_sch (KiCad schematic)
At the start: 98 parts, among them U1 ProMicro

Commit message: ven. 22 déc. 2023 01:02:29 CET
Parts:
- MX38: footprint _mx:MX-Alps-Hybrid-2.75U-ReversedStabilizers -> _mx:MX-Alps-Hybrid-2.75U
- MX39: footprint _mx:MX-Alps-Hybrid-2.25U-ReversedStabilizers -> _mx:MX-Alps-Hybrid-2.25U
Changed lines of the file:
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@@
       (effects (font (size 1.27 1.27)) (justify right) hide)
     )
-    (property "Footprint" "_mx:MX-Alps-Hybrid-2.75U-ReversedStabilizers" (at 63.5 121.92 0)
+    (property "Footprint" "_mx:MX-Alps-Hybrid-2.75U" (at 63.5 121.92 0)
       (effects (font (size 1.27 1.27)) hide)
     )
@@
       (effects (font (size 1.27 1.27)) (justify right) hide)
     )
-    (property "Footprint" "_mx:MX-Alps-Hybrid-2.25U-ReversedStabilizers" (at 71.12 121.92 0)
-      (effects (font (size 1.27 1.27)) hide)
-    )
+    (property "Footprint" "_mx:MX-Alps-Hybrid-2.25U" (at 71.12 121.92 0)
+      (effects (font (size 1.27 1.27)) hide)
+    )
