File: 007k/pcb/little/little.kicad_pcb (KiCad board)
At the start: 2 copper layers, 98 parts, among them U1 ProMicro

Commit message: ven. 22 déc. 2023 01:02:29 CET
Parts:
- added REF1: MountingHole_3.2mm_M3, MountingHole:MountingHole_3.2mm_M3, F.Cu at (120.1, 106.9)
- added REF2: MountingHole_3.2mm_M3, MountingHole:MountingHole_3.2mm_M3, F.Cu at (310.6, 106.9)
- added REF3: MountingHole_3.2mm_M3, MountingHole:MountingHole_3.2mm_M3, F.Cu at (220.1, 126.0)
- added REF4: MountingHole_3.2mm_M3, MountingHole:MountingHole_3.2mm_M3, F.Cu at (355.8, 147.4)
- added REF5: MountingHole_3.2mm_M3, MountingHole:MountingHole_3.2mm_M3, F.Cu at (124.8, 164.1)
- added REF6: MountingHole_3.2mm_M3, MountingHole:MountingHole_3.2mm_M3, F.Cu at (217.7, 165.6)
- added REF7: MountingHole_3.2mm_M3, MountingHole:MountingHole_3.2mm_M3, F.Cu at (311.8, 166.5)
- moved D38 21.9 mm to (175.9, 169.4), turned to 90 degrees
- moved D43 17.8 mm to (334.4, 153.6), turned to 90 degrees
- moved D39 14.4 mm to (259.5, 169.4), turned to 90 degrees
- moved D27 14.0 mm to (172.5, 148.9), turned to 90 degrees
- moved D28 14.0 mm to (191.5, 148.9), turned to 90 degrees
- moved D42 13.1 mm to (334.4, 172.7), turned to 90 degrees
- moved D44 13.1 mm to (353.4, 172.7), turned to 90 degrees
- moved D45 13.1 mm to (372.5, 172.7), turned to 90 degrees
- moved D30 7.09 mm to (248.7, 148.9), turned to 90 degrees
- moved D31 7.09 mm to (267.7, 148.9), turned to 90 degrees
- moved D29 7.09 mm to (229.6, 148.9), turned to 90 degrees
- moved D6 2.53 mm to (209.6, 116.5)
- moved D13 1.53 mm to (116.7, 135.5)
- moved D23 1.53 mm to (316.8, 135.5)
- moved D24 1.53 mm to (121.5, 154.6)
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Connections:
- U1 pad 1: COL7 -> unconnected-(U1-D3-TX-Pad1)
- U1 pad 10: COL3 -> L5
- U1 pad 11: COL2 -> L6
- U1 pad 12: COL1 -> L7
- U1 pad 18: L7 -> COL1
- U1 pad 19: L6 -> COL2
- U1 pad 2: COL6 -> L1
- U1 pad 20: L5 -> COL3
- U1 pad 21: L4 -> COL4
- U1 pad 22: L3 -> COL5
- U1 pad 23: L2 -> COL6
- U1 pad 24: L1 -> COL7
- U1 pad 7: unconnected-(U1-D4-Pad7) -> L2
- U1 pad 8: COL5 -> L3
- U1 pad 9: COL4 -> L4
Routing:
- net COL1: track 0.00 -> 458.8 mm
- net COL2: track 0.00 -> 435.8 mm
- net COL5: track 0.00 -> 420.8 mm
- net COL4: track 0.00 -> 404.9 mm
- net COL3: track 0.00 -> 364.6 mm
- net COL6: track 0.00 -> 350.9 mm
- net L7: track 0.00 -> 268.9 mm
- net L5: track 0.00 -> 236.2 mm, vias 0 -> 1
- net L1: track 0.00 -> 234.2 mm
- net L3: track 0.00 -> 231.5 mm
- net L8: track 0.00 -> 140.3 mm
- net L4: track 0.00 -> 117.0 mm
- net L2: track 0.00 -> 115.2 mm
- net L6: track 0.00 -> 114.8 mm, vias 0 -> 1
- net COL7: track 0.00 -> 98.2 mm
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- added copper zone on B.Cu, net GND
- added copper zone on F.Cu, net GND
Other:
- board outline added: 276.2 x 81 mm
- board text added: "007k"
- board text added: "Born to build"

Commit message: ven. 22 déc. 2023 11:54:46 CET
Other:
- board text removed: "007k"

Commit message: ven. 22 déc. 2023 21:50:38 CET
Parts:
- moved OLED1 1.09 mm to (349.8, 101.1)
Routing:
- net VCC: track 28.8 -> 29.9 mm
- net SCL: track 24.0 -> 25.1 mm
- net SDA: track 33.2 -> 34.3 mm

Commit message: sam. 23 déc. 2023 09:52:10 CET
Routing:
- net COL1: track 458.8 -> 474.5 mm
- net COL2: track 435.8 -> 448.1 mm
- net COL6: track 350.9 -> 340.3 mm
- net L8: track 140.3 -> 147.1 mm
- net COL4: track 404.9 -> 411.1 mm
- net L5: track 236.2 -> 242.0 mm, vias 1 -> 0
- net L7: track 268.9 -> 273.8 mm
- net L6: track 114.8 -> 110.2 mm, vias 1 -> 0
- net L3: track 231.5 -> 228.4 mm
- net L2: track 115.2 -> 112.8 mm
- net Net-(D30-A): track 13.0 -> 15.4 mm
- net L4: track 117.0 -> 118.7 mm
- net Net-(D43-A): track 8.63 -> 10.3 mm
- net COL3: track 364.6 -> 366.0 mm
- net COL5: track 420.8 -> 419.7 mm
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